Commit message: make table thicker

File: examples/models/fr3_algr_minimal_collision.urdf (robot description, URDF)
Before this commit: robot fr3_algr, 39 links, 39 joints
Links:
- link table: geometry collision box size=1.3208 1.8288 0.1; visual box size=1.3208 1.8288 0.1
Joints:
- joint table_joint: origin xyz=0.50165 0 -0.01 rpy=0 0 0 -> xyz=0.50165 0 -0.05 rpy=0 0 0
