Commit message: add feet with collisions

File: examples/models/harpy_planar.urdf (robot description, URDF)
Before this commit: robot harpy, 9 links, 9 joints
Links:
- added link FootLeft, mass 0.001; collision sphere radius=0.016; visual sphere radius=0.016
- added link FootRight, mass 0.001; collision sphere radius=0.016; visual sphere radius=0.016
- link TibiaLeft: mass 0.8 -> 0.1
- link TibiaRight: mass 0.8 -> 0.1
Joints:
- added joint TibiaLeft_FootLeft: type fixed, parent TibiaLeft, child FootLeft, origin xyz=0.0 0.0 -0.3 rpy=0.0 0.0 0.0, axis 0 1 0
- added joint TibiaRight_FootRight: type fixed, parent TibiaRight, child FootRight, origin xyz=0.0 0.0 -0.3 rpy=0.0 0.0 0.0, axis 0 1 0

Commit message: fix inertias

File: examples/models/harpy_planar.urdf (robot description, URDF)
Before this commit: robot harpy, 11 links, 11 joints
Links:
- link HipLeft: mass 1.0 -> 1
- link HipRight: mass 1.0 -> 1

Commit message: shuffle forward with trajopt

File: examples/models/harpy_planar.urdf (robot description, URDF)
Before this commit: robot harpy, 11 links, 11 joints
Links:
- added link ground, mass 1; collision box size=100 100 100
Joints:
- added joint world_ground: type fixed, parent world, child ground, origin xyz=0 0 0 rpy=0 0 0
