Commit message: simple harpy standing example

File: examples/models/harpy_2d.urdf (robot description, URDF)
Before this commit: robot harpy, 4 links, 4 joints
Links:
- link foot: geometry collision sphere radius=0.01; visual sphere radius=0.01

Commit message: harpy jumps on box example

File: examples/models/harpy_2d.urdf (robot description, URDF)
Before this commit: robot harpy_2d, 4 links, 4 joints
Links:
- added link box, mass 0.5; collision sphere radius=0.35; visual box size=0.5 0.5 0.5
Joints:
- added joint box_joint: type fixed, parent world, child box, origin xyz=1.2 0.0 0.25 rpy=0 0 0, axis 0 -1 0
