Commit message: simplify collision geoms

File: models/achilles/achilles.urdf (robot description, URDF)
Before this commit: robot achilles, 29 links, 28 joints
Links:
- link left_ankle_pitch: geometry collision sphere radius=0.02; collision sphere radius=0.02
- link right_ankle_pitch: geometry collision sphere radius=0.02; collision sphere radius=0.02
- link torso: geometry visual mesh filename=meshes/torso.obj
